Commit message: Add package

File: sim/pentos/urdf/pentos.urdf (robot description, URDF)
Before this commit: robot pentos, 7 links, 6 joints
Links:
- link a_axis: geometry collision mesh filename=package://pentos/meshes/A Axis.gltf scale=1 1 1; visual mesh filename=package://pentos/meshes/A Axis.gltf scale=1 1 1
- link b_axis: geometry collision mesh filename=package://pentos/meshes/B Axis.gltf scale=1 1 1; visual mesh filename=package://pentos/meshes/B Axis.gltf scale=1 1 1
- link frame: geometry collision mesh filename=package://pentos/meshes/Frame.gltf scale=1 1 1; visual mesh filename=package://pentos/meshes/Frame.gltf scale=1 1 1
- link x_carriage: geometry collision mesh filename=package://pentos/meshes/X Carriage.gltf scale=1 1 1; visual mesh filename=package://pentos/meshes/X Carriage.gltf scale=1 1 1
- link x_gantry: geometry collision mesh filename=package://pentos/meshes/X Gantry.gltf scale=1 1 1; visual mesh filename=package://pentos/meshes/X Gantry.gltf scale=1 1 1
- link y_gantry: geometry collision mesh filename=package://pentos/meshes/Y Gantry.gltf scale=1 1 1; visual mesh filename=package://pentos/meshes/Y Gantry.gltf scale=1 1 1
Joints:
- removed joint revolute_1_0
- removed joint revolute_2_0
- removed joint slider_1_0
- removed joint slider_2_0
- removed joint slider_3_0
- added joint a_axis_0: type continuous, parent y_gantry, child a_axis, origin xyz=-0.02 0.1 0.082 rpy=3.46945e-16 -4.66567e-16 -1.5708, axis -1 0 0
- added joint b_axis_0: type continuous, parent a_axis, child b_axis, origin xyz=0.1 -1.4456e-17 -0.047 rpy=-2.72712e-31 6.93889e-18 1.5708, axis 0 0 -1
- added joint x_axis_0: type prismatic, parent x_gantry, child x_carriage, origin xyz=0.165 0.005 0.02 rpy=0 -0 3.42114e-49, axis -1 0 0, limit lower=-10000 upper=10000 effort=1 velocity=1
- added joint y_axis_0: type prismatic, parent frame, child y_gantry, origin xyz=0.02 0.17 0.08 rpy=0 -0 1.98254e-16, axis 3.46945e-16 1 0, limit lower=-10000 upper=10000 effort=1 velocity=1
- added joint z_axis_0: type prismatic, parent frame, child x_gantry, origin xyz=-0.165 0.02 0.203 rpy=-6.50521e-17 5.78241e-17 -3.76158e-33, axis 0 0 -1, limit lower=-10000 upper=10000 effort=1 velocity=1
